Commit message: cleaned up code for ROS2 for beginners 2 final project

File: src/my_robot_description/urdf/arm.xacro (robot description, xacro)
@@ -80,5 +80,5 @@
         <parent link="base_link" />
         <child link="arm_base_link" />
-        <origin xyz="0 0 ${base_height}" rpy="0 0 0"/>
+        <origin xyz="${base_length/4.0} 0 ${base_height}" rpy="0 0 0"/>
     </joint>
 <!-- Gazebo Plugins for controlling the arm joints and publishing their states -->
@@ -99,12 +99,3 @@
         </plugin>
     </gazebo>
-      <!-- <gazebo>
-        <plugin filename="gz-sim-joint-state-publisher-system"
-                name="gz::sim::systems::JointStatePublisher"> -->
-        <!-- <joint_name>base_left_wheel_joint</joint_name>
-        <joint_name>base_right_wheel_joint</joint_name> -->
-        <!-- <joint_name>arm_base_forearm_joint</joint_name>
-        <joint_name>forearm_hand_joint</joint_name>
-        </plugin>
-    </gazebo> -->
 </robot>

File: src/my_robot_description/urdf/camera.xacro (robot description, xacro)
@@ -4,4 +4,5 @@
     <xacro:property name="camera_width" value="0.1" />
     <xacro:property name="camera_height" value="0.05" />
+<!-- Camera Link and Joint -->
     <link name="camera_link">
         <visual>
@@ -26,4 +27,5 @@
         <origin xyz="${base_length/2.0} 0 ${base_height/2.0}" rpy="0 0 0"/>
     </joint>
+<!-- Gazebo Camera Sensor -->
     <gazebo reference="camera_link">
         <sensor name="camera" type="camera">

File: src/my_robot_description/urdf/common_properties.xacro (robot description, xacro)
@@ -1,4 +1,5 @@
 <?xml version="1.0"?>
 <robot xmlns:xacro="http://www.ros.org/wiki/xacro">
+    <!-- Common material properties and Inertia macros -->
     <material name="blue">
         <color rgba="0 0 0.5 1" />

File: src/my_robot_description/urdf/mobile_base.xacro (robot description, xacro)
@@ -1,4 +1,5 @@
 <?xml version="1.0"?>
 <robot name="my_robot" xmlns:xacro="http://www.ros.org/wiki/xacro">
+<!-- Common Mobile Base Properties -->
     <xacro:property name="base_length" value="0.6" />
     <xacro:property name="base_width" value="0.4" />
@@ -7,4 +8,5 @@
     <xacro:property name="wheel_width" value="0.05" />
     <xacro:property name="caster_radius" value="0.05" />
+<!-- Mobile Base Links -->
     <link name="base_footprint"/>
     <link name="base_link">
@@ -76,4 +78,5 @@
                     o_xyz="0 0 -${wheel_radius / 2.0}" o_rpy="${-pi / 2.0} 0 0" />
     </link>
+<!-- Mobile Base Joints -->
     <joint name="base_joint" type="fixed">
         <parent link="base_footprint" />

File: src/my_robot_description/urdf/mobile_base_gazebo.xacro (robot description, xacro)
@@ -1,4 +1,5 @@
 <?xml version="1.0"?>
 <robot name="my_robot" xmlns:xacro="http://www.ros.org/wiki/xacro">
+<!-- Mobile Base Gazebo Plugins -->
     <gazebo reference="caster_wheel_link">
         <mu1 value="0.1"/>
